Commit message: add franka module

File: franka_description/urdf/effort_panda_arm.urdf.xacro (robot description, xacro)
@@ -1,27 +1,22 @@
 <?xml version='1.0' encoding='utf-8'?>
 <robot xmlns:xacro="http://www.ros.org/wiki/xacro" name="panda">
-  <xacro:arg name="arm_id" default="panda" /> <!-- Name of this panda -->
-  <xacro:arg name="hand" default="false" /> <!-- Should a franka_gripper be mounted at the flange?" -->
+  <xacro:arg name="arm_id" default="panda" /> <!-- argument로 변경 -->
+  <xacro:property name="arm_id" value="$(arg arm_id)" /> <!-- property 추가 -->
+  <xacro:arg name="hand" default="false" />
   <xacro:arg name="sim_ignition" default="false" />
   <xacro:arg name="use_fake_hardware" default="false" />
-  <xacro:arg name="simulation_controllers"
-    default="" />
-  <!-- initial position for simulations (Ignition) -->
+  <xacro:arg name="simulation_controllers" default="" />
   <xacro:arg name="initial_positions_file"
     default="$(find franka_description)/config/initial_positions.yaml" />
-  <!-- convert to property to use substitution in function -->
   <xacro:property name="initial_positions_file" default="$(arg initial_positions_file)" />
-  <link name="world">
-      </link>
+  ...
+  <!-- World link -->
+  <link name="world" />
   <joint name="world_base" type="fixed">
-    <origin
-      xyz="0 0 0"
-      rpy="0 0 0" />
-    <parent
-      link="world" />
-    <child
-      link="base" />
+    <origin xyz="0 0 0" rpy="0 0 0" />
+    <parent link="world" />
+    <child link="base" />
   </joint>
-  <!-- box shaped table as base -->
+  <!-- Base link (box shaped table) -->
   <link name="base">
     <visual>
@@ -43,6 +38,6 @@
       <mass value="10" />
       <inertia ixx="1e-3" ixy="0.0" ixz="0.0"
-        iyy="1e-3" iyz="0.0"
-        izz="1e-3" />
+               iyy="1e-3" iyz="0.0"
+               izz="1e-3" />
     </inertial>
   </link>
@@ -50,13 +45,12 @@
   <xacro:include filename="$(find franka_description)/urdf/panda_arm.xacro" />
   <xacro:panda_arm arm_id="$(arg arm_id)" sim_ignition="$(arg sim_ignition)" connected_to="base" xyz="0 0 1"
-    safety_distance="0.03" />
-  <!-- Panda gripper -->
+                   safety_distance="0.03" />
+  <!-- Panda hand (gripper) -->
   <xacro:if value="$(arg hand)">
-    <xacro:include filename="$(find franka_description)/urdf/hand.xacro" />
-    <xacro:hand ns="$(arg arm_id)" rpy="0 0 ${-pi/4}" connected_to="$(arg arm_id)_link8"
-      safety_distance="0.03" />
+    <xacro:include filename="$(find franka_description)/urdf/hand.xacro"/>
+    <xacro:hand ns="$(arg arm_id)" connected_to="${arm_id}_link8" rpy="0 0 ${-pi/4}" safety_distance="0.03"/>
   </xacro:if>
-  <xacro:include
-    filename="$(find franka_description)/urdf/ros2_control/effort_panda_arm.ros2_control.xacro" />
+  <!-- ROS2 control -->
+  <xacro:include filename="$(find franka_description)/urdf/ros2_control/effort_panda_arm.ros2_control.xacro" />
   <xacro:panda_arm_ros2_control
     ns="$(arg arm_id)"
@@ -64,13 +58,12 @@
     use_fake_hardware="$(arg use_fake_hardware)"
     initial_positions="${xacro.load_yaml(initial_positions_file)}" />
+  <!-- Ignition Gazebo plugin -->
   <xacro:if value="$(arg sim_ignition)">
-    <!-- Gazebo plugins -->
-    <gazebo reference="base">
-    </gazebo>
+    <gazebo reference="base"/>
     <gazebo>
       <plugin filename="ign_ros2_control-system" name="ign_ros2_control::IgnitionROS2ControlPlugin">
         <robot_param>robot_description</robot_param>
         <robot_param_node>robot_state_publisher</robot_param_node>
-        <parameters>$(find franka_gazebo)/config/franka_controllers.yaml</parameters>
+        <parameters>$(find franka_gazebo)/config/ros2_controllers.yaml</parameters>
       </plugin>
     </gazebo>

File: franka_description/urdf/effort_panda_arm_ft_sensor.urdf.xacro (robot description, xacro)
@@ -1,88 +1,35 @@
-<?xml version='1.0' encoding='utf-8'?>
+<?xml version="1.0"?>
 <robot xmlns:xacro="http://www.ros.org/wiki/xacro" name="panda">
-  <xacro:arg name="arm_id" default="panda" /> <!-- Name of this panda -->
-  <xacro:arg name="hand" default="false" /> <!-- Should a franka_gripper be mounted at the flange?" -->
-  <xacro:arg name="sim_ignition" default="false" />
-  <xacro:arg name="use_fake_hardware" default="false" />
-  <xacro:arg name="simulation_controllers"
-    default="" />
-  <!-- initial position for simulations (Ignition) -->
-  <xacro:arg name="initial_positions_file"
-    default="$(find franka_description)/config/initial_positions.yaml" />
-  <!-- convert to property to use substitution in function -->
-  <xacro:property name="initial_positions_file" default="$(arg initial_positions_file)" />
-  <link name="world">
-      </link>
-  <joint name="world_base" type="fixed">
-    <origin
-      xyz="0 0 0"
-      rpy="0 0 0" />
-    <parent
-      link="world" />
-    <child
-      link="base" />
+  <!-- ===================== -->
+  <!-- Arguments -->
+  <!-- ===================== -->
+  <xacro:arg name="use_sim_time" default="true"/>
+  <xacro:arg name="initial_positions_file" default="initial_positions.yaml"/>
+  <xacro:arg name="ros2_control_hardware_type" default="mock_components"/>
+  <!-- ===================== -->
+  <!-- World -->
+  <!-- ===================== -->
+  <link name="world"/>
+  <joint name="world_joint" type="fixed">
+    <parent link="world"/>
+    <child link="panda_link0"/>
   </joint>
-  <!-- box shaped table as base -->
-  <link name="base">
-    <visual>
-      <origin xyz="0 0 0.5" rpy="0 0 0" />
-      <geometry>
-        <box size="1.71 0.51 1" />
-      </geometry>
-      <material name="metal">
-        <color rgba="0.768627450980392 0.749019607843137 0.729411764705882 1" />
-      </material>
-    </visual>
-    <collision>
-      <origin xyz="0 0 0.5" rpy="0 0 0" />
-      <geometry>
-        <box size="1.71 0.51 1" />
-      </geometry>
-    </collision>
-    <inertial>
-      <mass value="10" />
-      <inertia ixx="1e-3" ixy="0.0" ixz="0.0"
-        iyy="1e-3" iyz="0.0"
-        izz="1e-3" />
-    </inertial>
-  </link>
-  <xacro:include filename="$(find franka_description)/urdf/box.urdf.xacro" />
-  <!-- Franka arm -->
-  <xacro:include filename="$(find franka_description)/urdf/panda_arm.xacro" />
-  <xacro:panda_arm arm_id="$(arg arm_id)" sim_ignition="$(arg sim_ignition)" connected_to="base" xyz="0 0 1"
-    safety_distance="0.03" />
-  <!-- Force torque sensor -->
-  <xacro:include filename="$(find franka_description)/urdf/ft_sensor.xacro" />
-  <xacro:ft_sensor ns="$(arg arm_id)" rpy="0 0 ${-pi/4}" connected_to="$(arg arm_id)_link8"
-    safety_distance="0.03" />
+  <!-- ===================== -->
+  <!-- Panda + Gripper (완성 URDF) -->
+  <!-- ===================== -->
+  <!-- ⚠️ 여기서 arm + hand + mesh 전부 포함됨 -->
   <xacro:include
-    filename="$(find franka_description)/urdf/ros2_control/effort_panda_arm.ros2_control.xacro" />
-  <xacro:panda_arm_ros2_control
-    ns="$(arg arm_id)"
-    sim_ignition="$(arg sim_ignition)"
-    use_fake_hardware="$(arg use_fake_hardware)"
-    initial_positions="${xacro.load_yaml(initial_positions_file)}" />
-  <xacro:if value="$(arg sim_ignition)">
-    <!-- Gazebo plugins -->
-    <gazebo reference="$(arg arm_id)_sensor_joint">
-      <sensor name="force_torque_sensor" type="force_torque">
-        <update_rate>100.0</update_rate>
-        <always_on>true</always_on>
-        <topic>/sensor_joint/force_torque</topic>
-        <visualize>true</visualize>
-        <ignition_frame_id>$(arg arm_id)_ft_sensor_link</ignition_frame_id>
-        <force_torque>
-          <frame>child</frame>
-          <measure_direction>child_to_parent</measure_direction>
-        </force_torque>
-      </sensor>
-    </gazebo>
-    <gazebo>
-      <plugin filename="ign_ros2_control-system" name="ign_ros2_control::IgnitionROS2ControlPlugin">
-        <robot_param>robot_description</robot_param>
-        <robot_param_node>robot_state_publisher</robot_param_node>
-        <parameters>$(find franka_gazebo)/config/franka_controllers.yaml</parameters>
-      </plugin>
-    </gazebo>
-  </xacro:if>
+    filename="$(find moveit_resources_panda_description)/urdf/panda.urdf"/>
+  <!-- ===================== -->
+  <!-- ros2_control -->
+  <!-- ===================== -->
+  <xacro:include filename="panda.ros2_control.xacro"/>
+  <xacro:include filename="panda_hand.ros2_control.xacro"/>
+  <xacro:panda_ros2_control
+      name="PandaFakeSystem"
+      initial_positions_file="$(arg initial_positions_file)"
+      ros2_control_hardware_type="$(arg ros2_control_hardware_type)"/>
+  <xacro:panda_hand_ros2_control
+      name="PandaHandFakeSystem"
+      ros2_control_hardware_type="$(arg ros2_control_hardware_type)"/>
 </robot>

File: franka_description/urdf/hand.xacro (robot description, xacro)
@@ -13,5 +13,5 @@
       <visual>
         <geometry>
-          <mesh filename="package://${description_pkg}/meshes/visual/hand.dae"/>
+          <mesh filename="$(find franka_description)/meshes/visual/hand.dae"/>
         </geometry>
       </visual>
@@ -52,4 +52,12 @@
         </geometry>
       </collision>
+      <!-- Inertial block added for hand -->
+      <inertial>
+        <mass value="0.73"/>
+        <origin xyz="0 0 0.06" rpy="0 0 0"/>
+        <inertia ixx="0.001" ixy="0" ixz="0"
+                 iyy="0.001" iyz="0"
+                 izz="0.001"/>
+      </inertial>
     </link>
     <!-- Define the hand_tcp frame -->
@@ -63,7 +71,21 @@
       <visual>
         <geometry>
-          <mesh filename="package://${description_pkg}/meshes/visual/finger.dae"/>
+          <mesh filename="$(find franka_description)/meshes/visual/finger.dae"/>
         </geometry>
       </visual>
+      <collision>
+        <origin xyz="0 0.015 0.022" rpy="0 0 0"/>
+        <geometry>
+          <box size="0.02 0.01 0.044"/>
+        </geometry>
+      </collision>
+      <!-- Inertial block added for left finger -->
+      <inertial>
+        <mass value="0.015"/>
+        <origin xyz="0 0.015 0.022" rpy="0 0 0"/>
+        <inertia ixx="1.875e-6" ixy="0" ixz="0"
+                 iyy="5e-7" iyz="0"
+                 izz="1.875e-6"/>
+      </inertial>
     </link>
     <link name="${ns}_rightfinger">
@@ -71,7 +93,20 @@
         <origin xyz="0 0 0" rpy="0 0 ${pi}"/>
         <geometry>
-          <mesh filename="package://${description_pkg}/meshes/visual/finger.dae"/>
+          <mesh filename="$(find franka_description)/meshes/visual/finger.dae"/>
         </geometry>
       </visual>
+      <collision>
+        <origin xyz="0 -0.015 0.022" rpy="0 0 0"/>
+        <geometry>
+          <box size="0.02 0.01 0.044"/>
+        </geometry>
+      </collision>
+      <inertial>
+        <mass value="0.015"/>
+        <origin xyz="0 -0.015 0.022" rpy="0 0 0"/>
+        <inertia ixx="1.875e-6" ixy="0" ixz="0"
+                 iyy="5e-7" iyz="0"
+                 izz="1.875e-6"/>
+      </inertial>
     </link>
     <joint name="${ns}_finger_joint1" type="prismatic">

File: franka_description/urdf/panda_arm.urdf.xacro (robot description, xacro)
@@ -2,5 +2,5 @@
 <robot xmlns:xacro="http://www.ros.org/wiki/xacro" name="panda">
   <xacro:arg name="arm_id" default="panda" /> <!-- Name of this panda -->
-  <xacro:arg name="hand" default="false" /> <!-- Should a franka_gripper be mounted at the flange?" -->
+  <xacro:arg name="hand" default="true" /> <!-- Should a franka_gripper be mounted at the flange?" -->
   <xacro:arg name="sim_ignition" default="false" />
   <xacro:arg name="use_fake_hardware" default="false" />
@@ -13,5 +13,5 @@
   <xacro:property name="initial_positions_file" default="$(arg initial_positions_file)" />
   <link name="world">
-      </link>
+  </link>
   <joint name="world_base" type="fixed">
     <origin
@@ -57,4 +57,5 @@
       safety_distance="0.03" />
   </xacro:if>
+  <!-- Arm ros2_control -->
   <xacro:include
     filename="$(find franka_description)/urdf/ros2_control/panda_arm.ros2_control.xacro" />
@@ -64,4 +65,10 @@
     use_fake_hardware="$(arg use_fake_hardware)"
     initial_positions="${xacro.load_yaml(initial_positions_file)}" />
+  <!-- Hand ros2_control -->
+  <xacro:if value="$(arg hand)">
+  <xacro:include filename="$(find franka_description)/urdf/panda_hand.ros2_control.xacro" />
+  <xacro:panda_hand_ros2_control
+    name="$(arg arm_id)_hand"
+    ros2_control_hardware_type="gz_sim" />  </xacro:if>
   <xacro:if value="$(arg sim_ignition)">
     <!-- Gazebo plugins -->
